Commit message: routine commit

File: arm_imitation/urdf/manipulator4.urdf (robot description, URDF)
Before this commit: robot mobile_manipulator, 10 links, 9 joints
Links:
- link elbow_motor: geometry collision mesh filename=package://mobile_manipulator/meshes/dynamixel_x64series.stl scale=0.001 0.001 0.001; visual mesh filename=package://mobile_manipulator/meshes/dynamixel_x64series.stl scale=0.001 0.001 0.001
- link shoulder_pitch_motor: geometry collision mesh filename=package://mobile_manipulator/meshes/dynamixel_x64series.stl scale=0.001 0.001 0.001; visual mesh filename=package://mobile_manipulator/meshes/dynamixel_x64series.stl scale=0.001 0.001 0.001
- link shoulder_roll_motor: geometry collision mesh filename=package://mobile_manipulator/meshes/dynamixel_x64series.stl scale=0.001 0.001 0.001; visual mesh filename=package://mobile_manipulator/meshes/dynamixel_x64series.stl scale=0.001 0.001 0.001
- link shoulder_yaw_motor: geometry collision mesh filename=package://mobile_manipulator/meshes/dynamixel_x64series.stl scale=0.001 0.001 0.001; visual mesh filename=package://mobile_manipulator/meshes/dynamixel_x64series.stl scale=0.001 0.001 0.001

File: arm_imitation/urdf/manipulator4.xacro (robot description, xacro)
@@ -40,5 +40,5 @@
       <origin xyz="${trans}" rpy="${rpy}"/>
       <geometry>
-        <box size="0.041 0.0402 0.0611"/>
+        <mesh filename="package://mobile_manipulator/meshes/dynamixel_x64series.stl" scale="0.001 0.001 0.001"/>
       </geometry>
     </collision>
