Commit message: routine commit

File: arm_imitation/urdf/manipulator3.xacro (robot description, xacro)
@@ -1,5 +1,4 @@
 <?xml version ="1.0"?>
-<robot xmlns:xacro="http://www.ros.org/wiki/xacro" name="manipulator">
-<!--0.5624 height to start-->
+<robot xmlns:xacro="http://www.ros.org/wiki/xacro" name="mobile_manipulator">
 <material name="white">
   <color rgba="1 1 1 1"/>
@@ -17,4 +16,5 @@
 <xacro:property name="LinkWidth" value="0.04"/>
 <xacro:property name="LinkHeight" value="0.04"/>
+<xacro:property name="LinkOverlapOffset" value="0.002"/>
 <xacro:property name="MXBracketLength" value="0.036"/>
 <xacro:property name="AXBracketLength" value="0.052"/>
@@ -44,4 +44,28 @@
     </collision>
 </xacro:macro>
+<xacro:macro name="AXInertial" params="trans rpy">
+  <inertial>
+    <origin xyz="${trans}" rpy="${rpy}"/>
+    <mass value="0.05573" />
+    <inertia ixx="0.00001611154" ixy="0.00000001397" ixz="0.0" iyy="0.00000888743" iyz="0.00000015948" izz="0.00001354172" />
+  </inertial>
+</xacro:macro>
+<xacro:macro name="AXVisual" params="trans rpy">
+  <visual>
+    <origin xyz="${trans}" rpy="${rpy}"/>
+    <geometry>
+      <mesh filename="package://mobile_manipulator/meshes/AX-12_18A - dynamixel_AXseries-1.stl" scale="0.001 0.001 0.001"/>
+    </geometry>
+    <material name="white"/>
+  </visual>
+</xacro:macro>
+<xacro:macro name="AXCollision" params="trans rpy">
+    <collision>
+      <origin xyz="${trans}" rpy="${rpy}"/>
+      <geometry>
+        <mesh filename="package://mobile_manipulator/meshes/AX-12_18A - dynamixel_AXseries-1.stl" scale="0.001 0.001 0.001"/>
+      </geometry>
+    </collision>
+</xacro:macro>
 <xacro:macro name="BracketInertial" params="trans rpy">
   <inertial>
@@ -103,5 +127,5 @@
     <origin xyz="${trans}" rpy="${rpy}"/>
     <geometry>
-      <box size="0.04 0.04 ${LinkLength}"/>
+      <box size="${LinkWidth} ${LinkHeight} ${LinkLength}"/>
     </geometry>
     <material name="white"/>
@@ -112,5 +136,5 @@
       <origin xyz="${trans}" rpy="${rpy}"/>
       <geometry>
-        <box size="0.04 0.04 ${LinkLength}"/>
+        <box size="${LinkWidth} ${LinkHeight} ${LinkLength}"/>
       </geometry>
     </collision>
@@ -133,9 +157,8 @@
 </xacro:macro>
 <!-- LINKS -->
-<!-- the trans parameter present here is to toggle distance of current object with respect to previous adjacent object i.e. its parent-->
   <link name="base_link">
-    <xacro:LinkInertial trans="0 0 0.5624" rpy="0 0 0" />
-    <xacro:LinkVisual trans="0 0 0.5624" rpy="0 0 0" />
-    <xacro:LinkCollision trans="0 0 0.5624" rpy="0 0 0" />
+    <xacro:LinkInertial trans="0 0 0" rpy="0 0 0" />
+    <xacro:LinkVisual trans="0 0 0" rpy="0 0 0" />
+    <xacro:LinkCollision trans="0 0 0" rpy="0 0 0" />
   </link>
   <link name="shoulder_yaw_motor">
@@ -144,9 +167,4 @@
     <xacro:MXCollision trans="0 0 ${MXDepth/2}" rpy="0 0 0"/>
   </link>
-  <link name="shoulder_roll_motor">
-  <xacro:MXInertial trans="0 ${MXLengthAxisLong} ${MXDepth/2 - MXWidth/2}" rpy="0 0 0 "/>
-  <xacro:MXVisual trans="0 ${MXLengthAxisLong} ${MXDepth/2 - MXWidth/2}" rpy="0 0 0 "/>
-  <xacro:MXCollision trans="0 ${MXLengthAxisLong} ${MXDepth/2 - MXWidth/2}" rpy="0 0 0"/>
-  </link>
   <link name="shoulder_pitch_motor">
     <xacro:MXInertial trans="0 ${MXLengthAxisLong} 0" rpy="0 0 0"/>
@@ -185,14 +203,12 @@
   </link>
  <!-- JOINTS -->
- <!-- the trans parameter present here is to toggle distance of current object with respect to next adjacent object i.e. its child-->
-  <xacro:FxdJoint id="base_joint" trans="0 ${LinkWidth/2} 0.5624" rpy="1.57 0 3.14" parent="base_link" child="shoulder_yaw_motor"/>
-  <xacro:RevJoint id="shoulder_yaw" trans="0 0 ${MXDepth}" rpy="1.57 0 0" parent="shoulder_yaw_motor" child="shoulder_roll_motor" axis="0 1 0" l="-3.14" u="3.14" v="1.0"/>
-  <xacro:RevJoint id="shoulder_roll" trans="0 ${MXLengthAxisLong} ${MXDepth/2}" rpy="1.57 0 1.57" parent="shoulder_roll_motor" child="shoulder_pitch_motor" axis="0 1 0" l="-3.14" u="3.14" v="1.0"/>
+ <!-- 1.57 0 3.14 -->
+  <xacro:FxdJoint id="base_joint" trans="0 ${LinkWidth/2} 0" rpy="1.57 0 3.14" parent="base_link" child="shoulder_yaw_motor"/>
+  <xacro:RevJoint id="shoulder_yaw" trans="0 0 ${MXDepth}" rpy="1.57 0 1.57" parent="shoulder_yaw_motor" child="shoulder_pitch_motor" axis="0 1 0" l="-3.14" u="3.14" v="1.0"/>
   <xacro:RevJoint id="shoulder_pitch" trans="0 ${MXLengthAxisLong} 0" rpy="0 1.57 1.57" parent="shoulder_pitch_motor" child="shoulder_bracket" axis="1 0 0" l="-1.57" u="1.57" v="1.0"/>
-  <!-- axis="1 0 0" l="-1.57" u="1.57" v="1.0" -->
-  <xacro:FxdJoint id="biceps_start" trans="0 0 ${MXBracketLength}" rpy="0 0 3.14" parent="shoulder_bracket" child="biscep"/>
+  <xacro:FxdJoint id="biceps_start" trans="0 0 ${MXBracketLength + LinkOverlapOffset}" rpy="0 0 3.14" parent="shoulder_bracket" child="biscep"/>
   <xacro:FxdJoint id="biceps_end" trans="0 0 ${LinkLength}" rpy="1.57 0 1.57" parent="biscep" child="elbow_motor"/>
   <xacro:RevJoint id="elbow_pitch" trans="0 ${MXLengthAxisLong} 0" rpy="0 1.57 1.57" parent="elbow_motor" child="elbow_bracket" axis="1 0 0" l="-1.57" u="1.57" v="1.0"/>
-  <xacro:FxdJoint id="forearm_start" trans="0 0 ${MXBracketLength}" rpy="0 0 3.14" parent="elbow_bracket" child="forearm"/>
+  <xacro:FxdJoint id="forearm_start" trans="0 0 ${MXBracketLength + LinkOverlapOffset}" rpy="0 0 3.14" parent="elbow_bracket" child="forearm"/>
   <xacro:FxdJoint id="forearm_end" trans="0 0 ${LinkLength}" rpy="1.57 0 1.57" parent="forearm" child="wrist_bracket"/>
 </robot>
