Commit message: routine commit

File: arm_imitation/urdf/manipulator4_meshed_test.urdf (robot description, URDF)
Before this commit: robot manipulator, 5 links, 4 joints
Joints:
- joint elbow_pitch: axis 1 0 0 -> -1 0 0

File: arm_imitation/urdf/manipulator4_meshed_test.xacro (robot description, xacro)
@@ -175,4 +175,4 @@
   <xacro:RevJoint id="shoulder_roll" trans="0 ${MXLengthAxisLong + MXDepth/2} ${MXLengthAxisLong}" rpy="1.57 1.57 3.14" parent="shoulder_roll_motor" child="shoulder_yaw_motor" axis="0 0 -1" l="-3.14" u="3.14" v="1.0"/>
   <xacro:RevJoint id="shoulder_yaw" trans="0 0 0" rpy="1.57 0 -1.57" parent="shoulder_yaw_motor" child="link_1" axis="1 0 0" l="-1.57" u="1.57" v="1.0"/>
-  <xacro:RevJoint id="elbow_pitch" trans="0 ${MXBracketLength + LinkLength + MXLengthAxisLong} 0" rpy="0 -1.57 0" parent="link_1" child="link_2" axis="1 0 0" l="-1.57" u="1.57" v="1.0"/>
+  <xacro:RevJoint id="elbow_pitch" trans="0 ${MXBracketLength + LinkLength + MXLengthAxisLong} 0" rpy="0 -1.57 0" parent="link_1" child="link_2" axis="-1 0 0" l="-1.57" u="1.57" v="1.0"/>
 </robot>
